File: SmartAPS.sch (KiCad schematic (older format))
At the start: 102 parts, among them M1 Mechanical-NC, M2 Mechanical-NC, M3 Mechanical-NC, M4 Mechanical, P1 12V IN, P2 GND, P3 OUT1, P4 OUT2, P5 USB_C_Receptacle_16P, P6 JESP32-DBG, Q1 MMBT5551, Q2 DMP3013SFV, Q3 MMBT5551, Q4 DMP3013SFV, Q5 MMBT5551, Q6 DMP3013SFV, Q7 TEMT6000X01, Q8 MMBT5551, U1 MCP1703T-3302E/MB, U2 MUN12AD01-SH, U3 INA226, U4 INA226, U5 IP6510, U6 INA226, U7 SHT20, U8 ESP32-WROOM-32U, U9 STM1001RWX6F

Commit message: Solve INA226/SHT20 address clash
Connections:
- net GND: no longer U3.1 (A1), U3.2 (A0)
- net SDA: now also U3.1 (A1), U3.2 (A0)
Other:
- note added: "AD = 0x4A\nWR = 0x94\nRD = 0x95"
- note removed: "AD = 0x40\nWR = 0x80\nRD = 0x81"
Changed lines of the file:
@@
 ALT1
 Text Notes 1100 3100 0    40   ~ 0
-AD = 0x40\nWR = 0x80\nRD = 0x81
+AD = 0x4A\nWR = 0x94\nRD = 0x95
 $Comp
 L BZ_Passive:R R22
@@
 Wire Wire Line
 	850  2650 850  2750
-Connection ~ 850  2850
-Wire Wire Line
-	850  2850 750  2850
-Connection ~ 850  2750
-Wire Wire Line
-	850  2750 850  2850
 Wire Wire Line
 	950  900  1000 900
@@
 	750  2500 750  2550
 Wire Wire Line
-	900  2850 850  2850
-Wire Wire Line
 	900  2550 750  2550
 Wire Wire Line
@@
 Wire Wire Line
 	9600 2750 9600 3100
+Wire Wire Line
+	750  2850 900  2850
+Wire Wire Line
+	850  2750 850  3100
+Wire Wire Line
+	850  3100 700  3100
+Connection ~ 850  2750
+Text Label 700  3100 0    50   ~ 0
+SDA
 $EndSCHEMATC

Commit message: Bug fixes, Remove SHT20
Parts:
- removed C22, C25: 0.1u, BZ_Capacitor:C_0603, symbol BZ_Passive:C
- removed TP4: GND, BZ_Misc:TE_RCT0805, symbol BZ_Misc:TP
- removed TP5: VDDA, BZ_Misc:TE_RCT0805, symbol BZ_Misc:TP
- removed TP8: SCL, BZ_Misc:TE_RCT0805, symbol BZ_Misc:TP
- removed TP9: SDA, BZ_Misc:TE_RCT0805, symbol BZ_Misc:TP
- removed U7: SHT20, BZ_Sensor:Sensirion_SHT20, symbol BZ_Sensor:Sensirion_SHT20
- added P7: Grove I2C, BZ_Connector:JST_S4B-PH-SM4-TB, symbol BZ_Connector:Header_01x04
- added R23, R24: 10K, BZ_Resistor:R_0603, symbol BZ_Passive:R
- renumbered C23 to C22, C24 to C23, C26 to C24, C27 to C25, C28 to C26, TP6 to TP4, TP7 to TP5, U8 to U7, U9 to U8
Connections:
- net SW1 is gone; now on net SW2: C20.2, S2.1, U7.6 (IO34)
- net 3V3: now also R23.1, R24.1
- net ALT1: now also U7.12 (IO27); no longer U7.11 (IO26)
- net BUZ: now also U7.10 (IO25); no longer U7.12 (IO27)
- net GND: now also P7.4 (Pin_4)
- net PWR1: now also U7.11 (IO26); no longer U7.10 (IO25)
- net SCL: now also P7.1 (Pin_1)
- net SDA: now also P7.2 (Pin_2)
- net SW2: now also R23.2; no longer C21.2, S3.1, U7.7 (IO35)
- net TCK: now also P6.4 (Pin_4); no longer P6.8 (Pin_8)
- net TDI: now also P6.8 (Pin_8); no longer P6.4 (Pin_4)
- net VDDA: now also P7.3 (Pin_3)
- net IR: no longer names the net of U7.24 (IO2)
- new net SW3: C21.2, R24.2, S3.1, U7.7 (IO35)
- no-connect marks 13 -> 14
Other:
- moved on the sheet: S1

Commit message: Change TEMT6000 output resistor to 100K
Parts:
- R17: value 10K -> 100K
Changed lines of the file:
@@
 P 1250 7100
 F 0 "R17" H 1298 7138 40  0000 L CNN
-F 1 "10K" H 1298 7062 40  0000 L CNN
+F 1 "100K" H 1298 7062 40  0000 L CNN
 F 2 "BZ_Resistor:R_0603" V 1180 7085 40  0001 C CNN
 F 3 "" H 1250 7085 40  0001 C CNN
