File: hw/SmartAPS.sch (KiCad schematic (older format))
At the start: 98 parts, among them M1 Mechanical-NC, M2 Mechanical-NC, M3 Mechanical-NC, M4 Mechanical, P1 12V IN, P2 GND, P3 OUT1, P4 OUT2, P5 USB_C_Receptacle_16P, P6 JESP32-DBG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

Commit message: Follow header name change
Parts:
- P1, P2: symbol BZ_Connector:Header_01x02 -> BZ_Connector:Conn_01x02
- P3, P4, P7: symbol BZ_Connector:Header_01x04 -> BZ_Connector:Conn_01x04
- P6: symbol BZ_Connector:Header_02x05 -> BZ_Connector:Conn_02x05
Changed lines of the file:
@@
 $EndComp
 $Comp
-L BZ_Connector:Header_01x02 P1
+L BZ_Connector:Conn_01x02 P1
 U 1 1 5E6687FD
 P 750 950
@@
 $EndComp
 $Comp
-L BZ_Connector:Header_01x04 P4
+L BZ_Connector:Conn_01x04 P4
 U 1 1 5EA818C1
 P 7050 2150
@@
 	10050 4150 10250 4150
 $Comp
-L BZ_Connector:Header_02x05 P6
+L BZ_Connector:Conn_02x05 P6
 U 1 1 5E63D243
-P 9750 3950
-F 0 "P6" H 9750 4250 40  0000 C CNN
-F 1 "JESP32-DBG" H 9800 3650 40  0000 C CNN
-F 2 "BZ_Connector:BHDR-THT-Vert-50mil_02x05" H 9750 3950 40  0001 C CNN
-F 3 "~" H 9750 3950 40  0001 C CNN
-	1    9750 3950
+P 9800 3950
+F 0 "P6" H 9800 4250 40  0000 C CNN
+F 1 "JESP32-DBG" H 9850 3650 40  0000 C CNN
+F 2 "BZ_Connector:BHDR-THT-Vert-50mil_02x05" H 9800 3950 40  0001 C CNN
+F 3 "~" H 9800 3950 40  0001 C CNN
+	1    9800 3950
 	1    0    0    -1
 $EndComp
@@
 	950  900  1000 900
 $Comp
-L BZ_Connector:Header_01x02 P2
+L BZ_Connector:Conn_01x02 P2
 U 1 1 5EE58F91
 P 750 1300
@@
 	3450 2100 3500 2100
 $Comp
-L BZ_Connector:Header_01x04 P3
+L BZ_Connector:Conn_01x04 P3
 U 1 1 5EB402BE
 P 3700 2150
@@
 	3900 5950 4150 5950
 $Comp
-L BZ_Connector:Header_01x04 P7
+L BZ_Connector:Conn_01x04 P7
 U 1 1 5EDC1433
 P 8600 5200

Commit message: Follow pin header name change
Parts:
- P6: footprint BZ_Connector:BHDR-THT-Vert-50mil_02x05 -> BZ_Connector:BOXHDR-THT-Vert-50mil-02x05
Changed lines of the file:
@@
 F 0 "P6" H 9800 4250 40  0000 C CNN
 F 1 "JESP32-DBG" H 9850 3650 40  0000 C CNN
-F 2 "BZ_Connector:BHDR-THT-Vert-50mil_02x05" H 9800 3950 40  0001 C CNN
+F 2 "BZ_Connector:BOXHDR-THT-Vert-50mil-02x05" H 9800 3950 40  0001 C CNN
 F 3 "~" H 9800 3950 40  0001 C CNN
 	1    9800 3950
